Commit message: Update robot.urdf.xacro

File: launch/include/config/robot.urdf.xacro (robot description, xacro)
@@ -25,5 +25,11 @@
     <parent link="chassis_link" />
     <child link="navsat_link" />
-    <origin xyz="0 0 0" rpy="0 0 0" />
+    <origin xyz="-0.30 0.30 -0.20" rpy="0 0 0" />
+  </joint>
+  <link name="gps"> </link>
+  <joint name="gps_joint" type="fixed">
+    <parent link="chassis_link" />
+    <child link="gps" />
+    <origin xyz="-0.30 0.30 -0.20" rpy="0 0 0" />
   </joint>
 </robot>
